Commit message: update

File: src/my_robot_model/description/imu.xacro (robot description, xacro)
@@ -12,5 +12,5 @@
       <pose>0 0 0 0 0 0</pose>
       <visualize>true</visualize>
-      <update_rate>15</update_rate>
+      <update_rate>13</update_rate>
       <always_on>true</always_on>
       <gz_frame_id>imu_link</gz_frame_id> <!-- `frame_id` in non-fortress -->
@@ -44,5 +44,5 @@
             <noise type="gaussian">
               <mean>0</mean>
-              <stddev>0.001</stddev>
+              <stddev>0.03</stddev>
             </noise>
           </x>
@@ -50,5 +50,5 @@
             <noise type="gaussian">
               <mean>0</mean>
-              <stddev>0.001</stddev>
+              <stddev>0.03</stddev>
             </noise>
           </y>
@@ -56,5 +56,5 @@
             <noise type="gaussian">
               <mean>0</mean>
-              <stddev>0.001</stddev>
+              <stddev>0.03</stddev>
             </noise>
           </z>

File: src/my_robot_model/description/lidar.xacro (robot description, xacro)
@@ -4,8 +4,8 @@
   <joint name="laser_joint" type="fixed">
     <parent link="chassis"/>
-    <child link="laser"/>
+    <child link="robot1_laser"/>
     <origin xyz="0 0 0.15" rpy="0 0 0"/>
   </joint>
-  <link name="laser">
+  <link name="robot1_laser">
     <visual>
       <geometry>
@@ -23,10 +23,11 @@
     </xacro:inertial_cylinder>
   </link>
-  <gazebo reference="laser">
+        s
+  <gazebo reference="robot1_laser">
     <sensor name="laser" type="gpu_lidar">
-      <topic>scan</topic>
-      <frame>laser</frame>
-      <update_rate>10</update_rate>
-      <gz_frame_id>laser</gz_frame_id>
+      <topic>/robot1/scan</topic>
+      <frame>robot1_laser</frame>
+      <update_rate>7</update_rate>
+      <gz_frame_id>robot1_laser</gz_frame_id>
       <lidar>
         <scan>

File: src/my_robot_model/description/robot_control.xacro (robot description, xacro)
@@ -54,4 +54,8 @@
       <publish_odom_tf>false</publish_odom_tf>
       <publish_wheel_tf>false</publish_wheel_tf>
+      <max_linear_acceleration>1.5</max_linear_acceleration>
+      <max_angular_acceleration>2.0</max_angular_acceleration>
+      <max_linear_velocity>1.5</max_linear_velocity>
+      <max_angular_velocity>2.5</max_angular_velocity>
     </plugin>
   </gazebo>

File: src/my_robot_model/description/robot_core.xacro (robot description, xacro)
@@ -70,6 +70,6 @@
       <friction>
         <ode>
-          <mu>1.0</mu>
-          <mu2>1.0</mu2>
+          <mu>2.0</mu>
+          <mu2>2.0</mu2>
         </ode>
       </friction>
@@ -81,6 +81,6 @@
 </link>
 <gazebo reference="left_wheel">
-  <mu1>1.0</mu1>
-  <mu2>1.0</mu2>
+  <mu1>2.0</mu1>
+  <mu2>2.0</mu2>
 </gazebo>
 <joint name="right_wheel_joint" type="continuous">
@@ -105,6 +105,6 @@
       <friction>
         <ode>
-          <mu>1.0</mu>
-          <mu2>1.0</mu2>
+          <mu>2.0</mu>
+          <mu2>2.0</mu2>
         </ode>
       </friction>
@@ -116,6 +116,6 @@
 </link>
 <gazebo reference="right_wheel">
-  <mu1>1.0</mu1>
-  <mu2>1.0</mu2>
+  <mu1>2.0</mu1>
+  <mu2>2.0</mu2>
 </gazebo>
 <joint name="caster_wheel_joint" type="fixed">
